File: NaD-main/Test_Project/Test_Project.kicad_pcb (KiCad board)
At the start: 2 copper layers, 40 parts, among them J1 SWD, J2 USART1, J3 3V3, J4 Barrel_Jack_Switch, J5 Screw_Terminal_01x02, SW1 SW_MEC_5E, SW2 SW_MEC_5E, U1 AMS1117-3.3, U2 STM32F103C8Tx, U3 L298HN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

Commit message: Documentation
Parts:
- removed J4: Barrel_Jack_Switch, Connector_BarrelJack:BarrelJack_GCT_DCJ200-10-A_Horizontal
- removed R5, R6: 10, Resistor_SMD:R_0805_2012Metric
- removed SW1, SW2: SW_MEC_5E, Button_Switch_THT:SW_PUSH_6mm
- D4, D5, D6, D7: footprint Diode_SMD:D_SMA -> Diode_SMD:D_0805_2012Metric
- U3: footprint Package_TO_SOT_THT:TO-220-15_P2.54x2.54mm_StaggerOdd_Lead4.58mm_Vertical -> Package_TO_SOT_THT:TO-220-15_P2.54x2.54mm_StaggerOdd_Lead5.84mm_TabDown
- moved D1 83.7 mm to (141.9, 133.2), turned to 0 degrees
- moved C1 83.3 mm to (142.6, 123.5)
- moved D2 81.8 mm to (121.5, 135.4), turned to 0 degrees
- moved J5 80.2 mm to (110.9, 125.5), turned to 90 degrees
- moved U1 79.7 mm to (132.4, 135.4), turned to 180 degrees
- moved D4 77.5 mm to (104.0, 129.7), turned to 90 degrees
- moved R1 74.1 mm to (119.2, 129.9), turned to 90 degrees
- moved D6 72.0 mm to (110.9, 133.3)
- moved C2 69.9 mm to (127.1, 124.5), turned to 180 degrees
- moved D5 67.9 mm to (103.2, 122.7), turned to 0 degrees
- moved U4 61.5 mm to (121.1, 92.8), turned to -90 degrees
- moved J2 59.6 mm to (144.6, 113.6), turned to 180 degrees
- moved U3 59.2 mm to (97.6, 126.7), turned to 90 degrees
- moved D7 58.1 mm to (110.8, 113.2), turned to 90 degrees
- moved C15 57.3 mm to (112.2, 86.8), turned to 180 degrees
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Connections:
- U2 pad 10: VCC -> unconnected-(U2-Pad10)
- U3 pad 10: IN3 -> unconnected-(U3-Pad10)
- U3 pad 12: IN4 -> unconnected-(U3-Pad12)
- U3 pad 9: +5V -> VCC
Routing:
- net IN4: track 115.5 -> 0.00 mm, vias 4 -> 0
- net IN3: track 95.1 -> 0.00 mm, vias 4 -> 0
- net GND: track 424.2 -> 329.7 mm, vias 25 -> 32
- net VCC: track 19.9 -> 95.7 mm, vias 2 -> 0
- net +5V: track 82.5 -> 9.87 mm
- net +3V3: track 217.4 -> 158.6 mm, vias 8 -> 9
- net Net-(R8-Pad1): track 39.4 -> 7.96 mm, vias 2 -> 0
- net IN2: track 111.2 -> 79.8 mm
- net Net-(R9-Pad1): track 46.8 -> 15.4 mm, vias 3 -> 0
- net Net-(D4-Pad2): track 52.3 -> 25.8 mm, vias 0 -> 1
- net ENA: track 40.9 -> 66.0 mm
- net Net-(D5-Pad2): track 45.1 -> 23.8 mm, vias 4 -> 1
- net DEBUG: track 3.78 -> 17.8 mm
- net NRST: track 7.03 -> 21.0 mm
- net OSC_IN: track 46.2 -> 32.5 mm, vias 2 -> 3
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